File: distortion-noise-and-ring-modulator-v1.2.brd (EAGLE design)
At the start: 46.7 x 24.1 mm, 77 parts, among them IC1 TL074JT, IC2 TL074JT, IC3 LM13700SL, Q1 MMBT3906, T1 NOISE-2N3904-DNM, U1 MC1496DR2G, X1 MA06-1JN-DNM, X2 MA06-1JN-DNM

Commit message: Tested and ready for production
Parts:
- R50: value 120k -> 100k
- R51: value 12k -> 10k
Routing:
- net N$9: track 30.8 -> 30.2 mm
- net GND: vias 26 -> 25
Changed lines of the file:
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@@
 <layer number="14" name="Route14" color="1" fill="6" visible="no" active="no"/>
 <layer number="15" name="Route15" color="4" fill="6" visible="no" active="no"/>
-<layer number="16" name="Bottom" color="1" fill="1" visible="no" active="yes"/>
+<layer number="16" name="Bottom" color="1" fill="1" visible="yes" active="yes"/>
 <layer number="17" name="Pads" color="2" fill="1" visible="yes" active="yes"/>
 <layer number="18" name="Vias" color="2" fill="1" visible="yes" active="yes"/>
@@
 <attribute name="VALUE" x="40.9575" y="14.2875" size="1.27" layer="27"/>
 </element>
-<element name="R50" library="rcl" library_urn="urn:adsk.eagle:library:334" package="R0402" package3d_urn="urn:adsk.eagle:package:23547/3" value="120k" x="34.6075" y="6.6675" smashed="yes">
+<element name="R50" library="rcl" library_urn="urn:adsk.eagle:library:334" package="R0402" package3d_urn="urn:adsk.eagle:package:23547/3" value="100k" x="34.6075" y="6.6675" smashed="yes">
 <attribute name="NAME" x="33.9725" y="7.3025" size="0.6096" layer="25" font="vector"/>
 <attribute name="POPULARITY" value="0" x="34.6075" y="6.6675" size="1.778" layer="27" display="off"/>
@@
 <attribute name="VALUE" x="33.9725" y="4.7625" size="1.27" layer="27"/>
 </element>
-<element name="R51" library="rcl" library_urn="urn:adsk.eagle:library:334" package="R0402" package3d_urn="urn:adsk.eagle:package:23547/3" value="12k" x="34.6075" y="5.476875" smashed="yes" rot="R180">
+<element name="R51" library="rcl" library_urn="urn:adsk.eagle:library:334" package="R0402" package3d_urn="urn:adsk.eagle:package:23547/3" value="10k" x="34.6075" y="5.476875" smashed="yes" rot="R180">
 <attribute name="NAME" x="33.9725" y="4.365625" size="0.6096" layer="25" font="vector"/>
 <attribute name="POPULARITY" value="0" x="34.6075" y="5.476875" size="1.778" layer="27" rot="R180" display="off"/>
@@
 <contactref element="R20" pad="2"/>
 <via x="24.13" y="4.60375" extent="1-16" drill="0.3302"/>
-<via x="14.9225" y="8.5725" extent="1-16" drill="0.3302"/>
 <wire x1="27.78125" y1="16.16875" x2="27.78125" y2="15.39875" width="0.254" layer="1"/>
 <via x="27.78125" y="15.39875" extent="1-16" drill="0.3302"/>
@@
 <wire x1="27.46375" y1="17.62125" x2="26.67" y2="17.62125" width="0.254" layer="1"/>
 <wire x1="26.67" y1="17.62125" x2="25.4" y2="17.62125" width="0.254" layer="1"/>
-<wire x1="21.59" y1="18.25625" x2="21.59" y2="17.93875" width="0.254" layer="1"/>
-<wire x1="20.79625" y1="17.36" x2="21.01125" y2="17.36" width="0.254" layer="1"/>
-<wire x1="21.59" y1="17.93875" x2="21.01125" y2="17.36" width="0.254" layer="1"/>
-<via x="21.59" y="18.25625" extent="1-16" drill="0.3302"/>
+<wire x1="20.79625" y1="17.36" x2="20.8525" y2="17.36" width="0.254" layer="1"/>
+<wire x1="21.74875" y1="17.78" x2="21.2725" y2="17.78" width="0.254" layer="1"/>
+<wire x1="21.2725" y1="17.78" x2="20.8525" y2="17.36" width="0.254" layer="1"/>
+<via x="21.74875" y="17.78" extent="1-16" drill="0.3302"/>
 <via x="24.13" y="17.62125" extent="1-16" drill="0.3302"/>
-<wire x1="24.13" y1="17.62125" x2="22.225" y2="17.62125" width="0.254" layer="16"/>
-<wire x1="22.225" y1="17.62125" x2="21.59" y2="18.25625" width="0.254" layer="16"/>
+<wire x1="24.13" y1="17.62125" x2="21.9075" y2="17.62125" width="0.254" layer="16"/>
+<wire x1="21.9075" y1="17.62125" x2="21.74875" y2="17.78" width="0.254" layer="16"/>
 <wire x1="33.5" y1="14.2875" x2="38.2625" y2="14.2875" width="0.254" layer="16"/>
 <wire x1="33.5" y1="14.2875" x2="30.6425" y2="17.145" width="0.254" layer="16"/>
@@
 <contactref element="IC1" pad="11"/>
 <contactref element="IC3" pad="6"/>
-<wire x1="31.4325" y1="10.795" x2="38.57625" y2="10.795" width="0.508" layer="1"/>
+<wire x1="31.4325" y1="10.795" x2="38.735" y2="10.795" width="0.508" layer="1"/>
 <contactref element="IC3" pad="13"/>
 <contactref element="IC3" pad="14"/>
@@
 <wire x1="38.735" y1="14.03" x2="38.735" y2="12.3825" width="0.254" layer="1"/>
 <via x="38.735" y="12.3825" extent="1-16" drill="0.3302"/>
-<via x="38.57625" y="10.795" extent="1-16" drill="0.3302"/>
+<via x="38.735" y="10.795" extent="1-16" drill="0.3302"/>
 <wire x1="46.0375" y1="6.64375" x2="45.9025" y2="6.50875" width="0.3556" layer="1"/>
 <wire x1="45.42625" y1="6.50875" x2="45.9025" y2="6.50875" width="0.3556" layer="1"/>
@@
 <wire x1="40.005" y1="12.7" x2="39.6875" y2="12.3825" width="0.254" layer="1"/>
 <wire x1="39.6875" y1="12.3825" x2="38.735" y2="12.3825" width="0.254" layer="1"/>
-<wire x1="38.735" y1="12.3825" x2="38.735" y2="10.95375" width="0.254" layer="16"/>
-<wire x1="38.735" y1="10.95375" x2="38.57625" y2="10.795" width="0.254" layer="16"/>
+<wire x1="38.735" y1="12.3825" x2="38.735" y2="10.795" width="0.254" layer="16"/>
 <wire x1="31.4325" y1="8.605" x2="31.4325" y2="10.795" width="0.3556" layer="1"/>
 <wire x1="40.64" y1="10.795" x2="41.275" y2="11.43" width="0.3556" layer="1"/>
 <wire x1="41.275" y1="11.43" x2="45.72" y2="11.43" width="0.3556" layer="1"/>
-<wire x1="38.57625" y1="10.795" x2="40.64" y2="10.795" width="0.3556" layer="1"/>
+<wire x1="38.735" y1="10.795" x2="40.64" y2="10.795" width="0.3556" layer="1"/>
 <wire x1="45.72" y1="11.43" x2="46.0375" y2="11.1125" width="0.3556" layer="1"/>
 <contactref element="R10" pad="2"/>
@@
 <wire x1="32.57375" y1="13.46125" x2="32.57375" y2="12.67" width="0.254" layer="1"/>
 <wire x1="32.57375" y1="12.67" x2="32.86125" y2="12.3825" width="0.254" layer="1"/>
-<wire x1="32.86125" y1="12.3825" x2="34.925" y2="12.3825" width="0.254" layer="1"/>
-<via x="34.925" y="12.3825" extent="1-16" drill="0.3302"/>
+<wire x1="32.86125" y1="12.3825" x2="35.56" y2="12.3825" width="0.254" layer="1"/>
+<via x="35.56" y="12.3825" extent="1-16" drill="0.3302"/>
 <wire x1="38.1" y1="9.8425" x2="35.56" y2="12.3825" width="0.254" layer="16"/>
-<wire x1="35.56" y1="12.3825" x2="34.925" y2="12.3825" width="0.254" layer="16"/>
 <wire x1="41.275" y1="10.4775" x2="41.275" y2="8.83" width="0.254" layer="1"/>
 <via x="41.275" y="10.4775" extent="1-16" drill="0.3302"/>

Commit message: Tested bom and gerber, v1.2
Parts:
- X1, X2: value MA06-1JN-DNM -> MA06-1JN
Changed lines of the file:
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@@
 <attribute name="VALUE" x="29.155" y="-2.045" size="1.27" layer="27"/>
 </element>
-<element name="X1" library="joakim" package="MA06N-1J" value="MA06-1JN-DNM" x="21.59" y="3.81" smashed="yes">
+<element name="X1" library="joakim" package="MA06N-1J" value="MA06-1JN" x="21.59" y="3.81" smashed="yes">
 <attribute name="VALUE" x="17.78" y="0.889" size="1.27" layer="27" ratio="10"/>
 </element>
-<element name="X2" library="joakim" package="MA06N-1J" value="MA06-1JN-DNM" x="21.59" y="19.05" smashed="yes" rot="R180">
+<element name="X2" library="joakim" package="MA06N-1J" value="MA06-1JN" x="21.59" y="19.05" smashed="yes" rot="R180">
 <attribute name="VALUE" x="25.4" y="21.971" size="1.27" layer="27" ratio="10" rot="R180"/>
 </element>
