File: distortion-noise-and-ring-modulator-v1.2.sch (EAGLE design)
At the start: 77 parts, among them IC1 TL074JT, IC2 TL074JT, IC3 LM13700SL, Q1 MMBT3906, T1 NOISE-2N3904-DNM, U1 MC1496DR2G, X1 MA06-1JN-DNM, X2 MA06-1JN-DNM

Commit message: Tested and ready for production
Parts:
- R50: value 120k -> 100k
- R51: value 12k -> 10k
Other:
- note removed: "TODO: TEST GAIN"
Changed lines of the file:
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@@
 <part name="GND25" library="supply1" library_urn="urn:adsk.eagle:library:371" deviceset="GND" device=""/>
 <part name="GND26" library="supply1" library_urn="urn:adsk.eagle:library:371" deviceset="GND" device=""/>
-<part name="R50" library="rcl" library_urn="urn:adsk.eagle:library:334" deviceset="R-EU_" device="R0402" package3d_urn="urn:adsk.eagle:package:23547/3" value="120k"/>
-<part name="R51" library="rcl" library_urn="urn:adsk.eagle:library:334" deviceset="R-EU_" device="R0402" package3d_urn="urn:adsk.eagle:package:23547/3" value="12k"/>
+<part name="R50" library="rcl" library_urn="urn:adsk.eagle:library:334" deviceset="R-EU_" device="R0402" package3d_urn="urn:adsk.eagle:package:23547/3" value="100k"/>
+<part name="R51" library="rcl" library_urn="urn:adsk.eagle:library:334" deviceset="R-EU_" device="R0402" package3d_urn="urn:adsk.eagle:package:23547/3" value="10k"/>
 <part name="GND3" library="supply1" library_urn="urn:adsk.eagle:library:371" deviceset="GND" device=""/>
 </parts>
@@
 - Using unneccesary input buffer op amp as output gain amp
 - Made card 2mm wider to accomodate additional resistors</text>
-<text x="167.64" y="63.5" size="3.81" layer="91">TODO: TEST GAIN</text>
 </plain>
 <instances>

Commit message: Tested bom and gerber, v1.2
Parts:
- X1, X2: value MA06-1JN-DNM -> MA06-1JN
Changed lines of the file:
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@@
 <part name="SUPPLY15" library="supply2" library_urn="urn:adsk.eagle:library:372" deviceset="-12V" device=""/>
 <part name="SUPPLY16" library="supply2" library_urn="urn:adsk.eagle:library:372" deviceset="+12V" device=""/>
-<part name="X1" library="joakim" deviceset="MA06-1J" device="N" value="MA06-1JN-DNM"/>
-<part name="X2" library="joakim" deviceset="MA06-1J" device="N" value="MA06-1JN-DNM"/>
+<part name="X1" library="joakim" deviceset="MA06-1J" device="N" value="MA06-1JN"/>
+<part name="X2" library="joakim" deviceset="MA06-1J" device="N" value="MA06-1JN"/>
 <part name="C3" library="rcl" library_urn="urn:adsk.eagle:library:334" deviceset="C-EU" device="C1206" package3d_urn="urn:adsk.eagle:package:23618/2" value="47uF"/>
 <part name="C2" library="rcl" library_urn="urn:adsk.eagle:library:334" deviceset="C-EU" device="C1206" package3d_urn="urn:adsk.eagle:package:23618/2" value="47uF"/>
